File: my node/node.sch (EAGLE design)
At the start: 23 parts, among them IC1 , J1 RF24, J4 FTDI, J5 I2C, J6 , J7 , J8 SPI, J9 I2C, U1 W25X40CL, U2 ATMEGA328P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

Commit message: Second version
Parts:
- added C7: 100nF, SparkFun-Capacitors:10UF-0805-10V-10%
- C1: value 100nF -> 10uF; device SparkFun-Capacitors:10UF-1206-6.3V-20% -> SparkFun-Capacitors:10UF-0805-10V-10%
- C2, C6: device SparkFun-Capacitors:10UF-1206-6.3V-20% -> SparkFun-Capacitors:10UF-0805-10V-10%
- renumbered IC1 to 662K, U1 to FLASH, U3 to ATSHA
Connections:
- net GND: now also C7.1
- net RXI: now also J4.TXO; no longer J4.RXI
- net TXO: now also J4.RXI; no longer J4.TXO
- net VCC: now also C7.2

Commit message: Third version
Fixed FTDI connectior
Pro Mini comatible pinout
Parts:
- removed J8: SPI, SparkFun-Connectors:AVR_SPI_PROG_3X2PTH
- removed J9: I2C, SparkFun-Connectors:CONN_04
- added C8: 100nF, SparkFun-Capacitors:10UF-0805-10V-10%
- added LED1: LED, led:LEDCHIP-LED0805
- added R6: 100Ohm, SparkFun-Resistors:0.22OHM-0805-1/4W-1%
- 662K: value (none) -> 662k
- ATSHA: value ATSHA204-TSU -> ATSHA
- C1: value 10uF -> 100nF
- FLASH: value W25X40CL -> SPI FLASH
- J4: value FTDI -> (none)
- J5: value I2C -> (none)
- R2, R3: value 10KOmh -> 10kOmh
- R4: value (none) -> 220k
- R5: value (none) -> 1MOhm
Connections:
- new net N$3: LED1.A, R6.1
- net A0: now also R4.2, R5.1
- net A2: now also R6.2; no longer R4.2, R5.1
- net GND: now also C8.2, LED1.C; no longer J8.6, J9.2
- net MISO: no longer J8.1
- net MOSI: no longer J8.4
- net RESET: no longer J8.5
- net SCK: no longer J8.3
- net SCL: no longer J9.3
- net SDA: no longer J9.4
- net VCC: now also C8.1; no longer J8.2, J9.1
Other:
- moved on the sheet: R4, R5
